File: at90can-uno/at90can-uno.kicad_pcb (KiCad board)
At the start: 2 copper layers, 68.6 x 53.3 mm, 8 parts, among them P1 Power, P2 Analog, P3 Digital, P4 Digital, P5 CONN_01X01, P6 CONN_01X01, P7 CONN_01X01, P8 CONN_01X01

Commit message: update to new kicad
Parts:
- added 1k1: R_Small, Resistor_SMD:R_0603_1608Metric_Pad1.05x0.95mm_HandSolder, F.Cu at (129.9, 103.0)
- added C1: 47uF, Capacitor_SMD:CP_Elec_6.3x5.4, F.Cu at (134.9, 111.3)
- added C10: 4.7uF, Capacitor_SMD:C_0603_1608Metric_Pad1.05x0.95mm_HandSolder, F.Cu at (246.7, 91.3)
- added C11: 100nF, Capacitor_SMD:C_0603_1608Metric_Pad1.05x0.95mm_HandSolder, F.Cu at (249.4, 54.9)
- added C12: 100nF, Capacitor_SMD:C_0603_1608Metric_Pad1.05x0.95mm_HandSolder, F.Cu at (234.2, 53.6)
- added C13: 4.7n, Capacitor_SMD:C_0603_1608Metric_Pad1.05x0.95mm_HandSolder, F.Cu at (118.6, 79.4)
- added C14: 100nF, Capacitor_SMD:C_0603_1608Metric_Pad1.05x0.95mm_HandSolder, F.Cu at (169.8, 106.9)
- added C15: 12pF, Capacitor_SMD:C_0603_1608Metric_Pad1.05x0.95mm_HandSolder, F.Cu at (142.4, 100.9)
- added C16: 12pF, Capacitor_SMD:C_0603_1608Metric_Pad1.05x0.95mm_HandSolder, F.Cu at (142.4, 93.3)
- added C2: 47uF, Capacitor_SMD:CP_Elec_5x5.4, F.Cu at (127.0, 110.6)
- added C3: 470pF, Capacitor_SMD:C_0603_1608Metric_Pad1.05x0.95mm_HandSolder, F.Cu at (118.6, 102.3)
- added C4: 2.2uF, Capacitor_Tantalum_SMD:CP_EIA-3216-18_Kemet-A, F.Cu at (119.0, 96.5)
- added C5: 33nF, Capacitor_SMD:C_0603_1608Metric_Pad1.05x0.95mm_HandSolder, F.Cu at (152.3, 95.2)
- added C6: 33nF, Capacitor_SMD:C_0603_1608Metric_Pad1.05x0.95mm_HandSolder, F.Cu at (161.5, 114.9)
- added C7: 100nF, Capacitor_SMD:C_0603_1608Metric_Pad1.05x0.95mm_HandSolder, F.Cu at (246.7, 93.8)
- added C8: 100nF, Capacitor_SMD:C_0603_1608Metric_Pad1.05x0.95mm_HandSolder, F.Cu at (127.1, 95.5)
- added C9: 100nF, Capacitor_SMD:C_0603_1608Metric_Pad1.05x0.95mm_HandSolder, F.Cu at (129.1, 95.3)
- added D1: D_Schottky_Small, Diode_SMD:D_SOD-123, F.Cu at (123.3, 81.5)
- added D2: D_Schottky_Small, Diode_SMD:D_SOD-123, F.Cu at (134.9, 123.2)
- added D3: LED_Small, LED_SMD:LED_0603_1608Metric_Pad1.05x0.95mm_HandSolder, F.Cu at (211.2, 95.9)
- added D4: LED_Small, LED_SMD:LED_0603_1608Metric_Pad1.05x0.95mm_HandSolder, F.Cu at (211.0, 91.6)
- added D5: NUP2105L, Package_TO_SOT_SMD:SOT-23, F.Cu at (180.8, 43.8)
- added D6: LED_Small, LED_SMD:LED_0603_1608Metric_Pad1.05x0.95mm_HandSolder, F.Cu at (129.9, 100.8)
- added F1: 200mA, Fuse:Fuse_0603_1608Metric_Pad1.05x0.95mm_HandSolder, F.Cu at (118.9, 84.5)
- added F2: 500mA, Fuse:Fuse_0603_1608Metric_Pad1.05x0.95mm_HandSolder, F.Cu at (129.4, 123.8)
- added FB1: Ferrite_Bead_Small, Inductor_SMD:L_0603_1608Metric_Pad1.05x0.95mm_HandSolder, F.Cu at (118.9, 81.5)
- added FB2: Ferrite_Bead_Small, Inductor_SMD:L_0603_1608Metric_Pad1.05x0.95mm_HandSolder, F.Cu at (132.0, 123.9)
- added J1: Barrel_Jack_Switch, Connector_BarrelJack:BarrelJack_Horizontal, F.Cu at (121.2, 118.7)
- added J2: USB_B_Micro, Connector_USB:USB_Micro-B_Amphenol_10103594-0001LF_Horizontal, F.Cu at (113.5, 88.3)
- added J3: Conn_01x04, Connector_JST:JST_GH_BM04B-GHS-TBT_1x04-1MP_P1.25mm_Vertical, F.Cu at (173.2, 48.9)
- added J4: Conn_01x04, Connector_JST:JST_GH_BM04B-GHS-TBT_1x04-1MP_P1.25mm_Vertical, F.Cu at (188.5, 51.4)
- added J5: Conn_01x04, Connector_JST:JST_SH_BM04B-SRSS-TB_1x04-1MP_P1.00mm_Vertical, B.Cu at (174.5, 81.9)
- added J6: AVR-JTAG-10, Connector_PinSocket_1.27mm:PinSocket_2x05_P1.27mm_Vertical, F.Cu at (167.6, 113.3)
- added J7: Conn_01x04, Connector_JST:JST_SH_BM04B-SRSS-TB_1x04-1MP_P1.00mm_Vertical, F.Cu at (174.5, 81.9)
- added J8: AVR-ISP-6, Connector_PinHeader_2.54mm:PinHeader_2x03_P2.54mm_Vertical, F.Cu at (174.5, 95.9)
- added JP1: SolderJumper_2_Bridged, Jumper:SolderJumper-2_P1.3mm_Bridged_Pad1.0x1.5mm, B.Cu at (175.4, 113.9)
- added JP2: SolderJumper_2_Bridged, Jumper:SolderJumper-2_P1.3mm_Bridged_Pad1.0x1.5mm, F.Cu at (196.7, 33.7)
- added JP3: SolderJumper_3_Open, Jumper:SolderJumper-3_P1.3mm_Open_Pad1.0x1.5mm_NumberLabels, F.Cu at (236.8, 46.4)
- added L1: 10uH, Inductor_SMD:L_0603_1608Metric_Pad1.05x0.95mm_HandSolder, F.Cu at (171.3, 108.3)
- added R1: 1k, Resistor_SMD:R_0603_1608Metric_Pad1.05x0.95mm_HandSolder, F.Cu at (217.4, 95.5)
- added R2: 1k, Resistor_SMD:R_0603_1608Metric_Pad1.05x0.95mm_HandSolder, F.Cu at (217.1, 92.0)
- added R3: 120R, Resistor_SMD:R_0603_1608Metric_Pad1.05x0.95mm_HandSolder, F.Cu at (185.9, 36.2)
- added R4: 1k5, Resistor_SMD:R_0603_1608Metric_Pad1.05x0.95mm_HandSolder, F.Cu at (148.3, 86.0)
- added R5: 1k5, Resistor_SMD:R_0603_1608Metric_Pad1.05x0.95mm_HandSolder, F.Cu at (146.5, 86.0)
- added R6: 1k5, Resistor_SMD:R_0603_1608Metric_Pad1.05x0.95mm_HandSolder, F.Cu at (243.5, 41.3)
- added R7: 1k5, Resistor_SMD:R_0603_1608Metric_Pad1.05x0.95mm_HandSolder, F.Cu at (229.5, 50.2)
- added R8: 10k, Resistor_SMD:R_0603_1608Metric_Pad1.05x0.95mm_HandSolder, F.Cu at (119.9, 75.6)
- added R9: 330R, Resistor_SMD:R_0603_1608Metric_Pad1.05x0.95mm_HandSolder, F.Cu at (117.3, 76.4)
- added SW1: SW_Push, Switches:TACTILE_SWITCH_SMD_6.0X3.5MM, F.Cu at (113.5, 78.1)
- added TP1: TestPoint, Connector_Pin:Pin_D0.7mm_L6.5mm_W1.8mm_FlatFork, F.Cu at (209.1, 132.2)
- added TP10: TestPoint, Connector_Pin:Pin_D0.7mm_L6.5mm_W1.8mm_FlatFork, F.Cu at (171.5, 117.7)
- added TP2: TestPoint, Connector_Pin:Pin_D0.7mm_L6.5mm_W1.8mm_FlatFork, F.Cu at (232.8, 112.5)
- added TP3: TestPoint, Connector_Pin:Pin_D0.7mm_L6.5mm_W1.8mm_FlatFork, B.Cu at (140.3, 86.9)
- added TP4: TestPoint, Connector_Pin:Pin_D0.7mm_L6.5mm_W1.8mm_FlatFork, B.Cu at (133.1, 81.0)
- added TP5: TestPoint, Connector_Pin:Pin_D0.7mm_L6.5mm_W1.8mm_FlatFork, F.Cu at (213.2, 128.5)
- added TP6: TestPoint, Connector_Pin:Pin_D0.7mm_L6.5mm_W1.8mm_FlatFork, B.Cu at (133.8, 97.1)
- added TP7: TestPoint, Connector_Pin:Pin_D0.7mm_L6.5mm_W1.8mm_FlatFork, F.Cu at (226.6, 124.2)
- added TP8: TestPoint, Connector_Pin:Pin_D0.7mm_L6.5mm_W1.8mm_FlatFork, B.Cu at (138.9, 90.0)
- added TP9: TestPoint, Connector_Pin:Pin_D0.7mm_L6.5mm_W1.8mm_FlatFork, B.Cu at (137.0, 100.3)
- added U1: AMS1117-5.0, Package_TO_SOT_SMD:SOT-223-3_TabPin2, F.Cu at (116.9, 108.4)
- added U2: MIC5205-3.3YM5, Package_TO_SOT_SMD:SOT-23-5, F.Cu at (116.6, 99.6)
- added U3: USBLC6-2SC6, Package_TO_SOT_SMD:SOT-23-6, F.Cu at (119.9, 88.3)
- added U4: FT232RL-REEL, digikey-footprints:SSOP-28_W5.30mm, F.Cu at (131.3, 88.3)
- added U5: AT90CAN64-16AU, Package_QFP:TQFP-64_14x14mm_P0.8mm, F.Cu at (156.8, 105.6)
- added U6: ISO1050DUB, Package_SO:SOP-8_6.62x9.15mm_P2.54mm, F.Cu at (202.4, 46.4)
- added U7: ISO1540, Package_SO:SOIC-8_3.9x4.9mm_P1.27mm, F.Cu at (241.8, 54.0)
- added Y1: Crystal_GND24_Small, Crystal:Crystal_SMD_3225-4Pin_3.2x2.5mm_HandSoldering, F.Cu at (142.4, 97.1)
Connections:
- P1 pad 3: /Reset -> #RST
- P1 pad 8: /Vin -> VIN
- P2 pad 1: /A0 -> ADC0
- P2 pad 2: /A1 -> ADC1
- P2 pad 3: /A2 -> ADC2
- P2 pad 4: /A3 -> ADC3
- P2 pad 5: /A4(SDA) -> TCK_ADC4
- P2 pad 6: /A5(SCL) -> TMS_ADC5
- P3 pad 1: /A5(SCL) -> SCL_INT0
- P3 pad 10: /8 -> OC1A
- P3 pad 2: /A4(SDA) -> SDA_INT1
- P3 pad 3: /AREF -> AREF
- P3 pad 5: /13(SCK) -> SCK
- P3 pad 6: /12(MISO) -> MISO
- P3 pad 7: /11(**/MOSI) -> MOSI
- P3 pad 8: /10(**/SS) -> #SS
- P3 pad 9: /9(**) -> OC1B
- P4 pad 1: /7 -> XCK0_AIN0
- P4 pad 2: /6(**) -> OC3A_AIN1
- P4 pad 3: /5(**) -> OC3B_INT4
- P4 pad 4: /4 -> OC2A
- P4 pad 5: /3(**) -> OC3C_INT5
- P4 pad 6: /2 -> T3_INT6
- P4 pad 7: /1(Tx) -> TXD1_INT3
- P4 pad 8: /0(Rx) -> RXD1_INT2
Routing:
- added copper zone on In2.Cu, net +5V
- added copper zone on In1.Cu, net GND
Other:
- copper layers 2 -> 4
- net class Default removed
